File: Sofle_v2_Choc/PCB/SofleKeyboard.sch (KiCad schematic (older format))
At the start: 84 parts, among them J2 4PIN, J3 OLED, P1 i2c_pin, P2 i2c_pin, SW1 SW_PUSH_LED, SW10 SW_PUSH_LED, SW11 SW_PUSH_LED, SW12 SW_PUSH_LED, SW13 SW_PUSH_LED, SW14 SW_PUSH_LED, SW15 SW_PUSH_LED, SW16 SW_PUSH_LED, SW17 SW_PUSH_LED, SW18 SW_PUSH_LED, SW19 SW_PUSH_LED, SW2 SW_PUSH_LED, SW20 SW_PUSH_LED, SW21 SW_PUSH_LED, SW22 SW_PUSH_LED, SW23 SW_PUSH_LED, SW24 SW_PUSH_LED, SW25 Rotary_Encoder_Switch, SW26 SW_PUSH_LED, SW27 SW_PUSH_LED, SW28 SW_PUSH_LED, SW29 SW_PUSH_LED, SW3 SW_PUSH_LED, SW30 SW_PUSH_LED, SW4 SW_PUSH_LED, SW5 SW_PUSH_LED, SW6 SW_PUSH_LED, SW7 SW_PUSH_LED, SW8 SW_PUSH_LED, SW9 SW_PUSH_LED, U1 ProMicro

Commit message: rename lib from SofleRGB to SofleChoc
Parts:
- SW1, SW10, SW11, SW12, SW13, SW14, SW15, SW16, SW17, SW18, SW19, SW2, SW20, SW21, SW22, SW23, SW24, SW26, SW27, SW28, SW29, SW3, SW30, SW4, SW5, SW6, SW7, SW8, SW9: footprint SofleRGB:Choc_Hotswap_SK6812MiniE -> SofleChoc:Choc_Hotswap_SK6812MiniE
